File: pcb_files/fightboard.kicad_pcb (KiCad board)
At the start: 2 copper layers, 233 x 74 mm, 29 parts, among them J1 SW_Push, K1 SW_Push, M1 XIAO-RP2040, P1 SW_Push, U1 SW_Push, U2 MCP23018-E_SP

Commit message: add finishing touches to prev design
Parts:
- added REF**: PinHeader_1x01_P2.54mm_Vertical, Connector_PinHeader_2.54mm:PinHeader_1x01_P2.54mm_Vertical, F.Cu at (166.0, 56.0)
- added REF**: PinHeader_1x01_P2.54mm_Vertical, Connector_PinHeader_2.54mm:PinHeader_1x01_P2.54mm_Vertical, F.Cu at (163.0, 66.0)
- added REF**: PinHeader_1x01_P2.54mm_Vertical, Connector_PinHeader_2.54mm:PinHeader_1x01_P2.54mm_Vertical, F.Cu at (108.0, 122.0)
- added REF**: PinHeader_1x01_P2.54mm_Vertical, Connector_PinHeader_2.54mm:PinHeader_1x01_P2.54mm_Vertical, F.Cu at (122.0, 122.0)
- added REF**: PinHeader_1x01_P2.54mm_Vertical, Connector_PinHeader_2.54mm:PinHeader_1x01_P2.54mm_Vertical, F.Cu at (163.0, 61.0)
- added REF**: PinHeader_1x01_P2.54mm_Vertical, Connector_PinHeader_2.54mm:PinHeader_1x01_P2.54mm_Vertical, F.Cu at (129.0, 122.0)
- added REF**: PinHeader_1x01_P2.54mm_Vertical, Connector_PinHeader_2.54mm:PinHeader_1x01_P2.54mm_Vertical, F.Cu at (115.0, 122.0)
- added REF**: PinHeader_1x01_P2.54mm_Vertical, Connector_PinHeader_2.54mm:PinHeader_1x01_P2.54mm_Vertical, F.Cu at (161.0, 56.0)
Routing:
- net unconnected-(U2-Pad15): track 0.00 -> 24.5 mm
- net unconnected-(U2-Pad16): track 0.00 -> 20.9 mm
- net unconnected-(U2-Pad18): track 0.00 -> 19.5 mm
- net unconnected-(M1-Pad10): track 0.00 -> 18.8 mm
- net unconnected-(U2-Pad19): track 0.00 -> 16.5 mm
- net unconnected-(M1-Pad9): track 0.00 -> 14.2 mm
- net unconnected-(M1-Pad8): track 0.00 -> 13.2 mm
- net unconnected-(M1-Pad11): track 0.00 -> 12.1 mm
- net Net-(BKSP1-Pad2): track 111.3 -> 115.4 mm
- net Net-(PLUS1-Pad2): track 84.8 -> 88.9 mm
- net Net-(ENTR1-Pad2): track 137.7 -> 141.8 mm
- net Net-(A1-Pad1): track 548.8 -> 552.1 mm
- net Net-(MNUS1-Pad2): track 54.0 -> 56.3 mm
- net Net-(M1-Pad12): track 80.4 -> 81.5 mm
Other:
- outline, holes or cut-outs redrawn
- board text added: "ADDR"
- board text added: "D10"
- board text added: "D7"
- board text added: "D8"
- board text added: "D9"
- board text added: "INT A"
- board text added: "INT B"
- board text added: "RESET"

Commit message: change enter to esc
Parts:
- renumbered ENTR1 to ESC1
Connections:
- ;1 pad 1: Net-(A1-Pad1) -> Net-(;1-Pad1)
- A1 pad 1: Net-(A1-Pad1) -> Net-(;1-Pad1)
- BKSP1 pad 1: Net-(A1-Pad1) -> Net-(;1-Pad1)
- D1 pad 1: Net-(A1-Pad1) -> Net-(;1-Pad1)
- ESC1 pad 1: Net-(A1-Pad1) -> Net-(;1-Pad1)
- I1 pad 1: Net-(A1-Pad1) -> Net-(;1-Pad1)
- J1 pad 1: Net-(A1-Pad1) -> Net-(;1-Pad1)
- K1 pad 1: Net-(A1-Pad1) -> Net-(;1-Pad1)
- L1 pad 1: Net-(A1-Pad1) -> Net-(;1-Pad1)
- M1 pad 13: Net-(A1-Pad1) -> Net-(;1-Pad1)
- MNUS1 pad 1: Net-(A1-Pad1) -> Net-(;1-Pad1)
- O1 pad 1: Net-(A1-Pad1) -> Net-(;1-Pad1)
- P1 pad 1: Net-(A1-Pad1) -> Net-(;1-Pad1)
- PLUS1 pad 1: Net-(A1-Pad1) -> Net-(;1-Pad1)
- S1 pad 1: Net-(A1-Pad1) -> Net-(;1-Pad1)
- U1 pad 1: Net-(A1-Pad1) -> Net-(;1-Pad1)
- U2 pad 1: Net-(A1-Pad1) -> Net-(;1-Pad1)
- W1 pad 1: Net-(A1-Pad1) -> Net-(;1-Pad1)
Routing:
- net Net-(A1-Pad1): track 552.1 -> 0.00 mm, vias 7 -> 0
- net Net-(;1-Pad1): track 0.00 -> 537.5 mm, vias 0 -> 7
Other:
- board text added: "ESC"
- board text removed: "ENTER"

Commit message: update pcb
Parts:
- removed the REF** at (166.0, 56.0)
- removed the REF** at (84.0, 62.0)
- removed the REF** at (163.0, 66.0)
- removed the REF** at (108.0, 122.0)
- removed the REF** at (122.0, 122.0)
- removed the REF** at (110.0, 62.0)
- removed the REF** at (163.0, 61.0)
- removed the REF** at (129.0, 122.0)
- removed the REF** at (115.0, 122.0)
- removed the REF** at (72.0, 62.0)
- removed the REF** at (98.0, 62.0)
- removed the REF** at (161.0, 56.0)
Connections:
- M1 pad 2: unconnected-(M1-Pad2) -> Net-(M1-Pad2)
- REF** pad 1: Net-(A1-Pad1) -> Net-(;1-Pad1)
- U2 pad 15: unconnected-(U2-Pad15) -> Net-(;1-Pad1)
- U2 pad 16: unconnected-(U2-Pad16) -> Net-(M1-Pad2)
Routing:
- net Net-(M1-Pad2): track 0.00 -> 73.5 mm
- net unconnected-(M1-Pad4): track 69.1 -> 0.00 mm
- net unconnected-(M1-Pad3): track 57.3 -> 0.00 mm
- net unconnected-(M1-Pad2): track 43.5 -> 0.00 mm
- net Net-(;1-Pad1): track 537.5 -> 569.3 mm, vias 7 -> 8
- net unconnected-(M1-Pad1): track 31.8 -> 0.00 mm
- net unconnected-(U2-Pad15): track 24.5 -> 0.00 mm
- net unconnected-(U2-Pad16): track 20.9 -> 0.00 mm
- net unconnected-(U2-Pad18): track 19.5 -> 0.00 mm
- net unconnected-(M1-Pad10): track 18.8 -> 0.00 mm
- net unconnected-(U2-Pad19): track 16.5 -> 0.00 mm
- net unconnected-(M1-Pad9): track 14.2 -> 0.00 mm
- net unconnected-(M1-Pad8): track 13.2 -> 0.00 mm
- net unconnected-(M1-Pad11): track 12.1 -> 0.00 mm
Other:
- board text removed: "ADDR"
- board text removed: "D0"
- board text removed: "D1"
- board text removed: "D10"
- board text removed: "D2"
- board text removed: "D3"
- board text removed: "D7"
- board text removed: "D8"
- board text removed: "D9"
- board text removed: "INT A"
- board text removed: "INT B"
- board text removed: "RESET"
