File: pcb_files/fightboard.kicad_sch (KiCad schematic)
At the start: 18 parts, among them J1 SW_Push, K1 SW_Push, M1 XIAO-RP2040, P1 SW_Push, U1 SW_Push, U2 MCP23018-E_SP

Commit message: change enter to esc
Parts:
- renumbered ENTR1 to ESC1
Changed lines of the file:
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@@
   (symbol (lib_id "Switch:SW_Push") (at 147.32 114.3 0) (unit 1)
     (in_bom yes) (on_board yes)
-    (property "Reference" "ENTR1" (id 0) (at 147.32 106.68 0))
+    (property "Reference" "ESC1" (id 0) (at 147.32 106.68 0))
     (property "Value" "SW_Push" (id 1) (at 147.32 109.22 0))
     (property "Footprint" "Button_Switch_THT:SW_PUSH_6mm" (id 2) (at 147.32 109.22 0)
@@
     )
     (path "/ebdbdeab-6689-4f95-82fa-42ee0f37d64c"
-      (reference "ENTR1") (unit 1) (value "SW_Push") (footprint "Button_Switch_THT:SW_PUSH_6mm")
+      (reference "ESC1") (unit 1) (value "SW_Push") (footprint "Button_Switch_THT:SW_PUSH_6mm")
     )
     (path "/aa2854a8-68d4-4b10-9c63-d731cef4b360"

Commit message: update pcb
Connections:
- net at ;1.1, A1.1, BKSP1.1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: now also U2.15 (ADDR)
- net at U2.16 (~{RESET}): now also M1.2 (D1)
Changed lines of the file:
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@@
   (junction (at 236.22 58.42) (diameter 0) (color 0 0 0 0)
   )
+  (junction (at 208.28 146.05) (diameter 0) (color 0 0 0 0)
+  )
   (junction (at 124.46 132.08) (diameter 0) (color 0 0 0 0)
   )
@@
   (junction (at 124.46 119.38) (diameter 0) (color 0 0 0 0)
   )
+  (wire (pts (xy 185.42 135.89) (xy 195.58 135.89))
+    (stroke (width 0) (type default) (color 0 0 0 0))
+  )
   (wire (pts (xy 156.21 110.49) (xy 156.21 105.41))
     (stroke (width 0) (type default) (color 0 0 0 0))
@@
     (stroke (width 0) (type default) (color 0 0 0 0))
   )
+  (wire (pts (xy 195.58 149.86) (xy 177.8 149.86))
+    (stroke (width 0) (type default) (color 0 0 0 0))
+  )
   (wire (pts (xy 156.21 87.63) (xy 152.4 87.63))
     (stroke (width 0) (type default) (color 0 0 0 0))
@@
     (stroke (width 0) (type default) (color 0 0 0 0))
   )
+  (wire (pts (xy 195.58 138.43) (xy 195.58 149.86))
+    (stroke (width 0) (type default) (color 0 0 0 0))
+  )
   (wire (pts (xy 190.5 68.58) (xy 182.88 68.58))
     (stroke (width 0) (type default) (color 0 0 0 0))
@@
     (stroke (width 0) (type default) (color 0 0 0 0))
   )
+  (wire (pts (xy 185.42 146.05) (xy 185.42 135.89))
+    (stroke (width 0) (type default) (color 0 0 0 0))
+  )
   (wire (pts (xy 160.02 123.19) (xy 160.02 113.03))
     (stroke (width 0) (type default) (color 0 0 0 0))
@@
     (stroke (width 0) (type default) (color 0 0 0 0))
   )
+  (wire (pts (xy 177.8 58.42) (xy 190.5 58.42))
+    (stroke (width 0) (type default) (color 0 0 0 0))
+  )
   (wire (pts (xy 162.56 132.08) (xy 162.56 118.11))
     (stroke (width 0) (type default) (color 0 0 0 0))
@@
     (stroke (width 0) (type default) (color 0 0 0 0))
   )
+  (wire (pts (xy 177.8 149.86) (xy 177.8 58.42))
+    (stroke (width 0) (type default) (color 0 0 0 0))
+  )
   (wire (pts (xy 162.56 118.11) (xy 195.58 118.11))
     (stroke (width 0) (type default) (color 0 0 0 0))
@@
     (stroke (width 0) (type default) (color 0 0 0 0))
   )
+  (wire (pts (xy 208.28 146.05) (xy 185.42 146.05))
+    (stroke (width 0) (type default) (color 0 0 0 0))
+  )
